File: cv-switch/cv-switch/cv-switch.kicad_sch (KiCad schematic)
At the start: 30 parts, among them J1 AudioJack2_SwitchT, J2 AudioJack2_SwitchT, J3 Conn_02x05_Odd_Even, SW1 SW_DPDT_x2, U1 TL072, U3 TL072

Commit message: Small fixes for cv-switch
Other:
- note added: "(use log)"
Changed lines of the file:
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@@
+		)
+	)
+	(text "(use log)"
+		(exclude_from_sim no)
+		(at 173.228 126.238 0)
+		(effects
+			(font
+				(size 1.27 1.27)
+			)
+		)
+	)
+	(text "(use log)"
+		(exclude_from_sim no)
+		(at 117.094 57.912 0)
+		(effects
+			(font
+				(size 1.27 1.27)
+			)
 		)
 	)
